Commit message: Changed mesh to not depend on herbpy

File: test_data/robots/bh280.urdf (robot description, URDF)
Before this commit: robot bh280, 9 links, 8 joints
Links:
- link /finger0_0: geometry 
- link /finger0_1: geometry 
- link /finger0_2: geometry 
- link /finger1_0: geometry 
- link /finger1_1: geometry 
- link /finger1_2: geometry 
- link /finger2_1: geometry 
- link /finger2_2: geometry 
- link /hand_base: geometry 
